File: hardware/kicad/totp-0.1.kicad_sch (KiCad schematic)
At the start: 0 parts

Commit message: Schematic: ERC clean
Parts:
- added J1: Conn_01x08, symbol Connector_Generic:Conn_01x08
- added J2: Conn_01x04, symbol Connector_Generic:Conn_01x04
- added SW1, SW2, SW3: SW_Push, symbol Switch:SW_Push
- added U1: XIAO-nRF52840-SMD, Seeed_XIAO:XIAO-nRF52840-DIP, symbol Seeed_XIAO:XIAO-nRF52840-SMD
Connections:
- new net +3V3: J1.1 (Pin_1), J2.2 (Pin_2), U1.12 (3V3_OUT)
- new net BTN_CONFIRM: SW3.1, U1.10 (D9)
- new net BTN_NEXT: SW1.1, U1.7 (D6)
- new net BTN_PREV: SW2.1, U1.8 (D7)
- new net EPD_BUSY: J1.8 (Pin_8), U1.1 (D0)
- new net EPD_CLK: J1.4 (Pin_4), U1.9 (D8)
- new net EPD_CS: J1.5 (Pin_5), U1.2 (D1)
- new net EPD_DC: J1.6 (Pin_6), U1.3 (D2)
- new net EPD_DIN: J1.3 (Pin_3), U1.11 (D10)
- new net EPD_RST: J1.7 (Pin_7), U1.4 (D3)
- new net GND: J1.2 (Pin_2), J2.1 (Pin_1), SW1.2, SW2.2, SW3.2, U1.13 (GND), U1.18 (GND), U1.20 (GND)
- new net I2C_SCL: J2.4 (Pin_4), U1.6 (D5)
- new net I2C_SDA: J2.3 (Pin_3), U1.5 (D4)
- no-connect marks 0 -> 7

Commit message: PCB: import footprints and rough placement, also fix erc rules with the duped pwr
Parts:
- J1: footprint (none) -> Connector_PinHeader_2.54mm:PinHeader_1x08_P2.54mm_Vertical
- J2: footprint (none) -> Connector_PinHeader_2.54mm:PinHeader_1x04_P2.54mm_Vertical
- SW1, SW2, SW3: footprint (none) -> Button_Switch_SMD:SW_SPST_PTS645Sx43SMTR92
Changed lines of the file:
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@@
 			)
 		)
-		(property "Footprint" ""
+		(property "Footprint" "Button_Switch_SMD:SW_SPST_PTS645Sx43SMTR92"
 			(at 97.79 82.55 0)
 			(hide yes)
@@
 			)
 		)
-		(property "Footprint" ""
+		(property "Footprint" "Button_Switch_SMD:SW_SPST_PTS645Sx43SMTR92"
 			(at 111.76 78.74 0)
 			(hide yes)
@@
 			)
 		)
-		(property "Footprint" ""
+		(property "Footprint" "Connector_PinHeader_2.54mm:PinHeader_1x04_P2.54mm_Vertical"
 			(at 127 40.64 0)
 			(hide yes)
@@
 			)
 		)
-		(property "Footprint" ""
+		(property "Footprint" "Connector_PinHeader_2.54mm:PinHeader_1x08_P2.54mm_Vertical"
 			(at 88.9 39.37 0)
 			(hide yes)
@@
 			)
 		)
-		(property "Footprint" ""
+		(property "Footprint" "Button_Switch_SMD:SW_SPST_PTS645Sx43SMTR92"
 			(at 129.54 76.2 0)
 			(hide yes)
